File: hardware/schematics/CAN_Node2pi.sch (EAGLE design)
At the start: 13 parts, among them IC1 MCP2515-E/P, Q2 BSS138, X1 FC-135FC-135, X2 FC-135FC-135

Commit message: changes to schematics
Parts:
- removed RPI-GPIO: OUT, pinhead:PINHD-2X20
- removed X1: FC-135FC-135, m-pad-2.1:FC-135FC-135
- added 3V3, 5V0, GND: IN, pinhead:PINHD-1X1
Connections:
- net N$12: now also IC1.OSC2; no longer X1.2
- net N$13: now also IC1.OSC1; no longer X1.1
- net N$15: now also 5V0.1
- net N$3: now also 3V3.1
- net N$5: now also GND.1
Changed lines of the file:
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@@
 <part name="CAN-HIGH" library="pinhead" deviceset="PINHD-1X1" device="" value="IN"/>
 <part name="CAN-LOW" library="pinhead" deviceset="PINHD-1X1" device="" value="IN"/>
-<part name="RPI-GPIO" library="pinhead" deviceset="PINHD-2X20" device="" value="OUT"/>
 <part name="U$2" library="mcp2561" deviceset="MCP2561" device="MCP"/>
 <part name="R3" library="rcl" deviceset="R-US_" device="M2309" value="600k"/>
@@
 <part name="R5" library="rcl" deviceset="R-US_" device="M2309" value="10k"/>
 <part name="R6" library="rcl" deviceset="R-US_" device="M2309" value="10k"/>
-<part name="X1" library="m-pad-2.1" deviceset="FC-135" device="FC-135"/>
 <part name="X2" library="m-pad-2.1" deviceset="FC-135" device="FC-135"/>
+<part name="5V0" library="pinhead" deviceset="PINHD-1X1" device="" value="IN"/>
+<part name="3V3" library="pinhead" deviceset="PINHD-1X1" device="" value="IN"/>
+<part name="GND" library="pinhead" deviceset="PINHD-1X1" device="" value="IN"/>
 </parts>
 <sheets>
 <sheet>
 <plain>
-<text x="154.94" y="111.76" size="1.778" layer="91">5V</text>
-<text x="154.94" y="106.68" size="1.778" layer="91">3V3</text>
-<text x="154.94" y="101.6" size="1.778" layer="91">GND</text>
+<text x="116.84" y="111.76" size="1.778" layer="91">5V</text>
+<text x="101.6" y="109.22" size="1.778" layer="91">3V3</text>
+<text x="185.42" y="101.6" size="1.778" layer="91">GND</text>
 </plain>
 <instances>
 <instance part="CAN-HIGH" gate="G$1" x="193.04" y="81.28"/>
 <instance part="CAN-LOW" gate="G$1" x="193.04" y="43.18"/>
-<instance part="RPI-GPIO" gate="A" x="33.02" y="68.58"/>
 <instance part="U$2" gate="G$1" x="147.32" y="76.2"/>
 <instance part="R3" gate="G$1" x="175.26" y="68.58" rot="R90"/>
@@
 <instance part="R5" gate="G$1" x="116.84" y="81.28" rot="R90"/>
 <instance part="R6" gate="G$1" x="101.6" y="76.2" rot="R270"/>
-<instance part="X1" gate="G$1" x="88.9" y="71.12"/>
 <instance part="X2" gate="G$1" x="88.9" y="71.12"/>
+<instance part="5V0" gate="G$1" x="35.56" y="121.92" rot="MR0"/>
+<instance part="3V3" gate="G$1" x="35.56" y="109.22" rot="MR0"/>
+<instance part="GND" gate="G$1" x="35.56" y="99.06" rot="MR0"/>
 </instances>
 <busses>
@@
 <segment>
 <pinref part="C1" gate="G$1" pin="2"/>
-<wire x1="185.42" y1="58.42" x2="185.42" y2="96.52" width="0.1524" layer="91"/>
-<wire x1="185.42" y1="96.52" x2="144.78" y2="96.52" width="0.1524" layer="91"/>
+<wire x1="185.42" y1="58.42" x2="185.42" y2="101.6" width="0.1524" layer="91"/>
+<wire x1="185.42" y1="101.6" x2="121.92" y2="101.6" width="0.1524" layer="91"/>
 <pinref part="U$2" gate="G$1" pin="VSS"/>
 <wire x1="129.54" y1="78.74" x2="121.92" y2="78.74" width="0.1524" layer="91"/>
@@
 <pinref part="IC1" gate="G$1" pin="VSS"/>
 <wire x1="121.92" y1="63.5" x2="83.82" y2="63.5" width="0.1524" layer="91"/>
-<wire x1="48.26" y1="101.6" x2="121.92" y2="101.6" width="0.1524" layer="91"/>
-<wire x1="121.92" y1="101.6" x2="144.78" y2="101.6" width="0.1524" layer="91"/>
-<wire x1="144.78" y1="101.6" x2="152.4" y2="101.6" width="0.1524" layer="91"/>
+<wire x1="45.72" y1="101.6" x2="121.92" y2="101.6" width="0.1524" layer="91"/>
 <wire x1="121.92" y1="78.74" x2="121.92" y2="101.6" width="0.1524" layer="91"/>
 <junction x="121.92" y="78.74"/>
 <junction x="121.92" y="101.6"/>
-<wire x1="144.78" y1="96.52" x2="144.78" y2="101.6" width="0.1524" layer="91"/>
-<junction x="144.78" y="101.6"/>
+<wire x1="45.72" y1="101.6" x2="45.72" y2="99.06" width="0.1524" layer="91"/>
+<pinref part="GND" gate="G$1" pin="1"/>
+<wire x1="45.72" y1="99.06" x2="38.1" y2="99.06" width="0.1524" layer="91"/>
 </segment>
 </net>
@@
 <pinref part="R6" gate="G$1" pin="1"/>
 <wire x1="101.6" y1="83.82" x2="101.6" y2="81.28" width="0.1524" layer="91"/>
-<wire x1="45.72" y1="106.68" x2="101.6" y2="106.68" width="0.1524" layer="91"/>
-<wire x1="101.6" y1="106.68" x2="152.4" y2="106.68" width="0.1524" layer="91"/>
-<wire x1="101.6" y1="83.82" x2="101.6" y2="106.68" width="0.1524" layer="91"/>
+<wire x1="38.1" y1="109.22" x2="101.6" y2="109.22" width="0.1524" layer="91"/>
+<wire x1="101.6" y1="83.82" x2="101.6" y2="109.22" width="0.1524" layer="91"/>
 <junction x="101.6" y="83.82"/>
-<junction x="101.6" y="106.68"/>
+<pinref part="3V3" gate="G$1" pin="1"/>
 </segment>
 </net>
@@
 <pinref part="R5" gate="G$1" pin="2"/>
 <wire x1="93.98" y1="93.98" x2="83.82" y2="93.98" width="0.1524" layer="91"/>
-<wire x1="43.18" y1="111.76" x2="93.98" y2="111.76" width="0.1524" layer="91"/>
 <wire x1="93.98" y1="111.76" x2="116.84" y2="111.76" width="0.1524" layer="91"/>
-<wire x1="116.84" y1="111.76" x2="152.4" y2="111.76" width="0.1524" layer="91"/>
 <wire x1="116.84" y1="86.36" x2="116.84" y2="111.76" width="0.1524" layer="91"/>
-<junction x="116.84" y="111.76"/>
 <wire x1="93.98" y1="93.98" x2="93.98" y2="111.76" width="0.1524" layer="91"/>
 <junction x="93.98" y="93.98"/>
+<pinref part="5V0" gate="G$1" pin="1"/>
+<wire x1="38.1" y1="121.92" x2="83.82" y2="121.92" width="0.1524" layer="91"/>
+<wire x1="83.82" y1="121.92" x2="83.82" y2="111.76" width="0.1524" layer="91"/>
+<wire x1="83.82" y1="111.76" x2="93.98" y2="111.76" width="0.1524" layer="91"/>
 <junction x="93.98" y="111.76"/>
 </segment>
@@
 <net name="N$12" class="0">
 <segment>
-<pinref part="X1" gate="G$1" pin="2"/>
 <pinref part="X2" gate="G$1" pin="2"/>
+<pinref part="IC1" gate="G$1" pin="OSC2"/>
+<wire x1="88.9" y1="68.58" x2="83.82" y2="68.58" width="0.1524" layer="91"/>
 </segment>
 </net>
 <net name="N$13" class="0">
 <segment>
-<pinref part="X1" gate="G$1" pin="1"/>
 <pinref part="X2" gate="G$1" pin="1"/>
+<pinref part="IC1" gate="G$1" pin="OSC1"/>
+<wire x1="83.82" y1="78.74" x2="88.9" y2="78.74" width="0.1524" layer="91"/>
+<wire x1="88.9" y1="78.74" x2="88.9" y2="76.2" width="0.1524" layer="91"/>
 </segment>
 </net>
